File: hardware/carrier/PigeonCarrier/PigeonCarrier.kicad_pcb (KiCad board)
At the start: 2 copper layers, 140.3 x 140.3 mm, 95 parts, among them J1 10164227-1001A1RLF, J2 10164227-1001A1RLF, J3 BATT CONN, Q1 CSD18540Q5B, Q2 CSD18540Q5B, U1 LM61495RPHR, U2 LM74502DDFR, U3 INA226AIDGSR, U4 TPS62933FDRLR, U5 3.3uH, U6 TLV75801PDRVR, U7 TLV75801PDRVR

Commit message: Update carrier schematics, parts library, and JLC rules
Parts:
- added C34: 1uF, PCM_JLCPCB:C_0603, F.Cu at (267.0, 54.8)
- added C35: 1uF, PCM_JLCPCB:C_0603, F.Cu at (267.0, 57.0)
- added C36: 100nF, PCM_JLCPCB:C_0402, F.Cu at (240.0, 52.2)
- added C37: 10uF, Capacitor_SMD:C_1210_3225Metric, F.Cu at (221.2, 20.9)
- added C47: 10uF, Capacitor_SMD:C_1210_3225Metric, F.Cu at (221.2, 25.1)
- added C48: 100nF, PCM_JLCPCB:C_0402, F.Cu at (231.1, 31.0)
- added C49: 100nF, PCM_JLCPCB:C_0402, F.Cu at (231.1, 32.9)
- added C50: 100nF, PCM_JLCPCB:C_0402, F.Cu at (231.1, 34.7)
- added C51: 100nF, PCM_JLCPCB:C_0402, F.Cu at (231.1, 36.6)
- added C52: 10uF, Capacitor_SMD:C_1210_3225Metric, F.Cu at (221.2, 29.4)
- added C53: 10uF, Capacitor_SMD:C_1210_3225Metric, F.Cu at (221.2, 33.6)
- added C54: 10uF, Capacitor_SMD:C_1210_3225Metric, F.Cu at (221.2, 37.9)
- added C55: 10uF, Capacitor_SMD:C_1210_3225Metric, F.Cu at (226.8, 20.9)
- added C56: 10uF, Capacitor_SMD:C_1210_3225Metric, F.Cu at (226.8, 25.1)
- added C57: 10uF, Capacitor_SMD:C_1210_3225Metric, F.Cu at (226.8, 29.4)
- added C58: 100nF, PCM_JLCPCB:C_0402, F.Cu at (247.2, 34.0)
- added C59: 100nF, PCM_JLCPCB:C_0402, F.Cu at (247.2, 35.9)
- added C60: 100nF, PCM_JLCPCB:C_0402, F.Cu at (247.2, 37.7)
- added C61: 100nF, PCM_JLCPCB:C_0402, F.Cu at (247.2, 39.6)
- added J301: FH12-22S-0.5SH(55), PigeonVision:Hirose_FH12-22S-0.5SH_1x22-1MP_P0.50mm_Horizontal, F.Cu at (256.0, 50.4)
- added J302: FH12-22S-0.5SH(55), PigeonVision:Hirose_FH12-22S-0.5SH_1x22-1MP_P0.50mm_Horizontal, F.Cu at (256.0, 59.4)
- added J401: A70-112-331N126, PigeonVision:RJ45_EDAC_A70-112-331N126, F.Cu at (228.5, 58.5)
- added J5: PJ-102AH, PigeonVision:SameSky_PJ-102AH_Horizontal, F.Cu at (260.5, 24.3)
- added L2: 6.8uH, JLCImport_Auto:CYA1040-6_8UH, F.Cu at (236.7, 24.4)
- added R103: 10, PigeonVision:KiCad_Resistor_SMD_R_0402_1005Metric, F.Cu at (250.0, 39.2)
- added R104: 10, PigeonVision:KiCad_Resistor_SMD_R_0402_1005Metric, F.Cu at (250.0, 41.2)
- added R15: 470Ω, PCM_JLCPCB:R_0402, F.Cu at (240.0, 54.0)
- added R16: 470Ω, PCM_JLCPCB:R_0402, F.Cu at (240.0, 55.9)
- added R17: 10kΩ, PCM_JLCPCB:R_0402, F.Cu at (231.1, 38.4)
- added R18: 15kΩ, PCM_JLCPCB:R_0402, F.Cu at (231.1, 40.3)
- added R19: 2.2kΩ, PCM_JLCPCB:R_0603, F.Cu at (266.9, 48.0)
- added R24: 0Ω, PCM_JLCPCB:R_0402, F.Cu at (231.1, 42.1)
- added R26: 47kΩ, PCM_JLCPCB:R_0402, F.Cu at (231.1, 44.0)
- added R27: 220Ω, PCM_JLCPCB:R_0402, F.Cu at (270.6, 19.7)
- added R28: 0Ω, PCM_JLCPCB:R_0603, F.Cu at (253.3, 39.3)
- added R29: 2.2kΩ, PCM_JLCPCB:R_0603, F.Cu at (266.9, 50.3)
- added R30: 2.2kΩ, PCM_JLCPCB:R_0603, F.Cu at (266.9, 52.5)
- added TP5: GND, TestPoint:TestPoint_Pad_D2.0mm, F.Cu at (267.2, 20.8)
- added TP6: GND, TestPoint:TestPoint_Pad_D2.0mm, F.Cu at (267.2, 24.8)
- added TP7: GND, TestPoint:TestPoint_Pad_D2.0mm, F.Cu at (267.2, 28.9)
- added U10: BMP581, PigeonVision:Bosch_BMP581_LGA-10_2x2mm_P0.5mm, F.Cu at (253.4, 42.2)
- added U6: TPD4EUSB30DQAR, PigeonVision:TI_DQA0010A_USON-10_1x2.5mm_P0.5mm, F.Cu at (240.2, 49.1)
- added U7: TPD4EUSB30DQAR, PigeonVision:TI_DQA0010A_USON-10_1x2.5mm_P0.5mm, F.Cu at (243.4, 49.1)
- added U8: TPS62933FDRLR, PigeonVision:SOT-583-8, F.Cu at (234.3, 32.1)
- added U9: BMI088, PigeonVision:Bosch_LGA-16_4.5x3mm_P0.5mm_LayoutBorder7x1y_ClockwisePinNumbering, F.Cu at (251.7, 35.9)
- TP4: value 4V_CAM -> 3V3_CAM
Connections:
- net Net-(U2-EN/UVLO) renamed /Power & Regulators/PWR_EN
- C3 pad 1: +3V3 -> 3V3_CM5
- J1 pad 1: unconnected-(J1-GND-Pad1) -> GND
- J1 pad 10: unconnected-(J1-Ethernet_Pair0_N-Pad10) -> /CM5/ETH0_N
- J1 pad 100: unconnected-(J1-CAM_GPIO1-Pad100) -> /CM5/CAM1_RST
- J1 pad 11: unconnected-(J1-Ethernet_Pair2_P-Pad11) -> /CM5/ETH2_P
- J1 pad 12: unconnected-(J1-Ethernet_Pair0_P-Pad12) -> /CM5/ETH0_P
- J1 pad 13: unconnected-(J1-GND-Pad13) -> GND
- J1 pad 14: unconnected-(J1-GND-Pad14) -> GND
- J1 pad 15: unconnected-(J1-Ethernet_nLED3(3.3v)-Pad15) -> /CM5/ETH_LED_K
- J1 pad 17: unconnected-(J1-Ethernet_nLED2(3.3v)-Pad17) -> /CM5/ETH_LED_G
- J1 pad 2: unconnected-(J1-GND-Pad2) -> GND
- J1 pad 22: unconnected-(J1-GND-Pad22) -> GND
- J1 pad 23: unconnected-(J1-GND-Pad23) -> GND
- J1 pad 3: unconnected-(J1-Ethernet_Pair3_P-Pad3) -> /CM5/ETH3_P
- J1 pad 32: unconnected-(J1-GND-Pad32) -> GND
- J1 pad 33: unconnected-(J1-GND-Pad33) -> GND
- J1 pad 35: unconnected-(J1-ID_SC-Pad35) -> /CM5/CAM1_I2C_SCL
- J1 pad 36: unconnected-(J1-ID_SD-Pad36) -> /CM5/CAM1_I2C_SDA
- J1 pad 4: unconnected-(J1-Ethernet_Pair1_P-Pad4) -> /CM5/ETH1_P
- J1 pad 42: unconnected-(J1-GND-Pad42) -> GND
- J1 pad 43: unconnected-(J1-GND-Pad43) -> GND
- J1 pad 5: unconnected-(J1-Ethernet_Pair3_N-Pad5) -> /CM5/ETH3_N
- J1 pad 50: unconnected-(J1-GPIO17-Pad50) -> /CM5/5V_RF_EN
- J1 pad 52: unconnected-(J1-GND-Pad52) -> GND
- J1 pad 53: unconnected-(J1-GND-Pad53) -> GND
- J1 pad 56: unconnected-(J1-GPIO3-Pad56) -> /Sensors/SENSOR_I2C_SCL
- J1 pad 58: unconnected-(J1-GPIO2-Pad58) -> /Sensors/SENSOR_I2C_SDA
- J1 pad 59: unconnected-(J1-GND-Pad59) -> GND
- J1 pad 6: unconnected-(J1-Ethernet_Pair1_N-Pad6) -> /CM5/ETH1_N
- J1 pad 60: unconnected-(J1-GND-Pad60) -> GND
- J1 pad 65: unconnected-(J1-GND-Pad65) -> GND
- J1 pad 66: unconnected-(J1-GND-Pad66) -> GND
- J1 pad 7: unconnected-(J1-GND-Pad7) -> GND
- J1 pad 71: unconnected-(J1-GND-Pad71) -> GND
- J1 pad 74: unconnected-(J1-GND-Pad74) -> GND
- J1 pad 77: unconnected-(J1-+5v_(Input)-Pad77) -> 5V_MAIN
- J1 pad 78: unconnected-(J1-GPIO_VREF(1.8v/3.3v_Input)-Pad78) -> 3V3_CM5
- J1 pad 79: unconnected-(J1-+5v_(Input)-Pad79) -> 5V_MAIN
- J1 pad 8: unconnected-(J1-GND-Pad8) -> GND
- J1 pad 80: unconnected-(J1-SCL0-Pad80) -> /CM5/CAM0_I2C_SCL
- J1 pad 81: unconnected-(J1-+5v_(Input)-Pad81) -> 5V_MAIN
- J1 pad 82: unconnected-(J1-SDA0-Pad82) -> /CM5/CAM0_I2C_SDA
- J1 pad 83: unconnected-(J1-+5v_(Input)-Pad83) -> 5V_MAIN
- J1 pad 84: unconnected-(J1-+3.3v_(Output)-Pad84) -> 3V3_CM5
- J1 pad 85: unconnected-(J1-+5v_(Input)-Pad85) -> 5V_MAIN
- J1 pad 86: unconnected-(J1-+3.3v_(Output)-Pad86) -> 3V3_CM5
- J1 pad 87: unconnected-(J1-+5v_(Input)-Pad87) -> 5V_MAIN
- J1 pad 9: unconnected-(J1-Ethernet_Pair2_N-Pad9) -> /CM5/ETH2_N
- J1 pad 97: unconnected-(J1-CAM_GPIO0-Pad97) -> /CM5/CAM0_RST
- J1 pad 98: unconnected-(J1-GND-Pad98) -> GND
- J2 pad 13: unconnected-(J2-GND-Pad13) -> GND
- J2 pad 14: unconnected-(J2-GND-Pad14) -> GND
- J2 pad 15: unconnected-(J2-MIPI0_D0_N-Pad15) -> /CM5/MIPI0_D0_N
- J2 pad 17: unconnected-(J2-MIPI0_D0_P-Pad17) -> /CM5/MIPI0_D0_P
- J2 pad 19: unconnected-(J2-GND-Pad19) -> GND
- J2 pad 20: unconnected-(J2-GND-Pad20) -> GND
- J2 pad 21: unconnected-(J2-MIPI0_D1_N-Pad21) -> /CM5/MIPI0_D1_N
- J2 pad 23: unconnected-(J2-MIPI0_D1_P-Pad23) -> /CM5/MIPI0_D1_P
- J2 pad 25: unconnected-(J2-GND-Pad25) -> GND
- J2 pad 26: unconnected-(J2-GND-Pad26) -> GND
- J2 pad 27: unconnected-(J2-MIPI0_C_N-Pad27) -> /CM5/MIPI0_CLK_N
- J2 pad 29: unconnected-(J2-MIPI0_C_P-Pad29) -> /CM5/MIPI0_CLK_P
- J2 pad 31: unconnected-(J2-GND-Pad31) -> GND
- J2 pad 32: unconnected-(J2-GND-Pad32) -> GND
- J2 pad 33: unconnected-(J2-MIPI0_D2_N-Pad33) -> /CM5/MIPI0_D2_N
- J2 pad 35: unconnected-(J2-MIPI0_D2_P-Pad35) -> /CM5/MIPI0_D2_P
- J2 pad 37: unconnected-(J2-GND-Pad37) -> GND
- J2 pad 38: unconnected-(J2-GND-Pad38) -> GND
- J2 pad 39: unconnected-(J2-MIPI0_D3_N-Pad39) -> /CM5/MIPI0_D3_N
- J2 pad 41: unconnected-(J2-MIPI0_D3_P-Pad41) -> /CM5/MIPI0_D3_P
- J2 pad 44: unconnected-(J2-GND-Pad44) -> GND
- J2 pad 50: unconnected-(J2-GND-Pad50) -> GND
- J2 pad 55: unconnected-(J2-GND-Pad55) -> GND
- J2 pad 56: unconnected-(J2-GND-Pad56) -> GND
- J2 pad 61: unconnected-(J2-GND-Pad61) -> GND
- J2 pad 62: unconnected-(J2-GND-Pad62) -> GND
- J2 pad 67: unconnected-(J2-GND-Pad67) -> GND
- J2 pad 68: unconnected-(J2-GND-Pad68) -> GND
- J2 pad 7: unconnected-(J2-GND-Pad7) -> GND
- J2 pad 73: unconnected-(J2-GND-Pad73) -> GND
- J2 pad 74: unconnected-(J2-GND-Pad74) -> GND
- J2 pad 75: unconnected-(J2-MIPI1_D0_N-Pad75) -> /CM5/MIPI1_D0_N
- J2 pad 77: unconnected-(J2-MIPI1_D0_P-Pad77) -> /CM5/MIPI1_D0_P
- J2 pad 79: unconnected-(J2-GND-Pad79) -> GND
- J2 pad 8: unconnected-(J2-GND-Pad8) -> GND
- J2 pad 80: unconnected-(J2-GND-Pad80) -> GND
- J2 pad 81: unconnected-(J2-MIPI1_D1_N-Pad81) -> /CM5/MIPI1_D1_N
- J2 pad 83: unconnected-(J2-MIPI1_D1_P-Pad83) -> /CM5/MIPI1_D1_P
- J2 pad 85: unconnected-(J2-GND-Pad85) -> GND
- J2 pad 86: unconnected-(J2-GND-Pad86) -> GND
- J2 pad 87: unconnected-(J2-MIPI1_C_N-Pad87) -> /CM5/MIPI1_CLK_N
- J2 pad 89: unconnected-(J2-MIPI1_C_P-Pad89) -> /CM5/MIPI1_CLK_P
- J2 pad 91: unconnected-(J2-GND-Pad91) -> GND
- J2 pad 92: unconnected-(J2-GND-Pad92) -> GND
- J2 pad 93: unconnected-(J2-MIPI1_D2_N-Pad93) -> /CM5/MIPI1_D2_N
- J2 pad 94: unconnected-(J2-MIPI1_D3_N-Pad94) -> /CM5/MIPI1_D3_N
- J2 pad 95: unconnected-(J2-MIPI1_D2_P-Pad95) -> /CM5/MIPI1_D2_P
- J2 pad 96: unconnected-(J2-MIPI1_D3_P-Pad96) -> /CM5/MIPI1_D3_P
- J2 pad 97: unconnected-(J2-GND-Pad97) -> GND
- J2 pad 98: unconnected-(J2-GND-Pad98) -> GND
- R11 pad 2: /Power & Regulators/VBAT->5V_RF/5V_RF_EN -> /CM5/5V_RF_EN
- TP4 pad 1: 4V_CAM -> 3V3_CAM
- U3 pad 4: /Power & Regulators/SDA_0 -> /Sensors/SENSOR_I2C_SDA
- U3 pad 5: /Power & Regulators/SCL_0 -> /Sensors/SENSOR_I2C_SCL
- U3 pad 6: +3V3 -> 3V3_CM5
- U4 pad 2: /Power & Regulators/VBAT->5V_RF/5V_RF_EN -> /CM5/5V_RF_EN
Other:
- copper layers 2 -> 4

Commit message: update updategit statusgit status
Parts:
- removed the C34 at (267.0, 54.8)
- removed the C34 at (191.3, 111.9)
- removed the C35 at (200.3, 122.3)
- removed the C35 at (267.0, 57.0)
- removed the C36 at (240.0, 52.2)
- removed the C36 at (169.5, 84.8)
- removed the C37 at (193.3, 115.1)
- removed the C37 at (221.2, 20.9)
- removed C4: 100nF, PCM_JLCPCB:C_0402
- removed J301, J302: FH12-22S-0.5SH(55), PigeonVision:Hirose_FH12-22S-0.5SH_1x22-1MP_P0.50mm_Horizontal
- removed J401: A70-112-331N126, PigeonVision:RJ45_EDAC_A70-112-331N126
- removed L1, L2: 6.8uH, JLCImport_Auto:CYA1040-6_8UH
- removed LED1, LED2, LED3: 0805G_Green, JLCImport_Auto:0805G_Green
- removed R103, R104: 10, PigeonVision:KiCad_Resistor_SMD_R_0402_1005Metric
- removed the R15 at (168.3, 80.5)
- removed the R15 at (240.0, 54.0)
- removed the R16 at (170.1, 80.5)
- removed the R16 at (240.0, 55.9)
- removed the R17 at (172.0, 80.5)
- removed the R17 at (231.1, 38.4)
- removed the R18 at (196.1, 112.0)
- removed the R18 at (231.1, 40.3)
- removed the R19 at (173.0, 86.2)
- removed the R19 at (266.9, 48.0)
- removed the R20 at (195.2, 112.0)
- removed the R20 at (177.3, 50.0)
- removed the R24 at (231.1, 42.1)
- removed the R24 at (191.5, 59.5)
- removed the R27 at (270.6, 19.7)
- removed the R27 at (187.5, 55.1)
- removed the U6 at (240.2, 49.1)
- removed the U6 at (196.9, 121.9)
- removed the U7 at (243.4, 49.1)
- removed the U7 at (193.3, 111.9)
- removed U8: TPS62933FDRLR, PigeonVision:SOT-583-8
- added C34: 10uF, Capacitor_SMD:C_1210_3225Metric, F.Cu at (111.5, 120.7)
- added C35: 10uF, Capacitor_SMD:C_1210_3225Metric, F.Cu at (111.5, 124.9)
- added C36: 10uF, Capacitor_SMD:C_1210_3225Metric, F.Cu at (111.5, 129.2)
- added C37: 10uF, Capacitor_SMD:C_1210_3225Metric, F.Cu at (111.5, 133.4)
- added C62: 10uF, Capacitor_SMD:C_1210_3225Metric, F.Cu at (183.3, 96.5)
- added C63: 10uF, Capacitor_SMD:C_1210_3225Metric, F.Cu at (183.3, 100.7)
- added C64: 10uF, Capacitor_SMD:C_1210_3225Metric, F.Cu at (188.9, 83.7)
- added C65: 10uF, Capacitor_SMD:C_1210_3225Metric, F.Cu at (188.9, 88.0)
- added C66: 10uF, Capacitor_SMD:C_1210_3225Metric, F.Cu at (188.9, 92.2)
- added C67: 100nF, PCM_JLCPCB:C_0402, F.Cu at (178.6, 127.3)
- added J10: USB4105_GF_A, PigeonVision:USB_C_Receptacle_GCT_USB4105_GF_A_16P, F.Cu at (183.0, 121.7)
- added J11: Samtec_TSM-102-01-L-SV-P-TR, PigeonVision:Samtec_TSM-102-01_SV_1x02_P2.54mm_SMD, F.Cu at (192.2, 120.3)
- added J4: BM04B-SRSS-TB(LF)(SN), PigeonVision:JST_SH_BM04B-SRSS-TB_1x04-1MP_P1.00mm_Vertical, F.Cu at (142.9, 83.8)
- added J7: FH12-22S-0.5SH(55), PigeonVision:Hirose_FH12-22S-0.5SH_1x22-1MP_P0.50mm_Horizontal, F.Cu at (161.7, 119.9)
- added J8: FH12-22S-0.5SH(55), PigeonVision:Hirose_FH12-22S-0.5SH_1x22-1MP_P0.50mm_Horizontal, F.Cu at (161.7, 128.9)
- added J9: A70-112-331N126, PigeonVision:RJ45_EDAC_A70-112-331N126, F.Cu at (162.7, 67.8)
- added Q3: BSS138BK,215, PigeonVision:Nexperia_SOT23_BSS138BK, F.Cu at (187.5, 133.9)
- added R15: 10, PigeonVision:KiCad_Resistor_SMD_R_0402_1005Metric, F.Cu at (156.9, 142.4)
- added R16: 10, PigeonVision:KiCad_Resistor_SMD_R_0402_1005Metric, F.Cu at (156.9, 144.4)
- added R17: 0Ω, PCM_JLCPCB:R_0603, F.Cu at (160.2, 142.5)
- added R18: 470Ω, PCM_JLCPCB:R_0402, F.Cu at (174.3, 63.3)
- added R19: 470Ω, PCM_JLCPCB:R_0402, F.Cu at (174.3, 65.2)
- added R20: 0Ω, PCM_JLCPCB:R_0402, F.Cu at (121.4, 122.6)
- added R24: 4.99kΩ, PCM_JLCPCB:R_0603, F.Cu at (121.8, 139.7)
- added R27: 51kΩ, PCM_JLCPCB:R_0402, F.Cu at (193.9, 68.2)
- added R31: 0Ω, PCM_JLCPCB:R_0402, F.Cu at (193.2, 91.8)
- added R32: 47kΩ, PCM_JLCPCB:R_0402, F.Cu at (193.2, 93.6)
- added R33: 15kΩ, PCM_JLCPCB:R_0402, F.Cu at (193.2, 95.5)
- added R34: 5.1kΩ, PCM_JLCPCB:R_0402, F.Cu at (178.6, 129.2)
- added R35: 5.1kΩ, PCM_JLCPCB:R_0402, F.Cu at (178.6, 131.0)
- added R36: 1kΩ, PCM_JLCPCB:R_0402, F.Cu at (178.6, 132.9)
- added R37: 10kΩ, PCM_JLCPCB:R_0402, F.Cu at (178.6, 134.7)
- added R38: 10kΩ, PCM_JLCPCB:R_0402, F.Cu at (178.6, 136.6)
- added SW1: PTS636 SK25 SMTR LFS, PigeonVision:CK_PTS636_SK25_SMTR_LFS_GullWing_SMD, F.Cu at (185.3, 129.0)
- added U11: TPD4E05U06DQAR, PigeonVision:TI_DQA0010A_USON-10_1x2.5mm_P0.5mm, F.Cu at (191.5, 133.8)
- added U12: TPD1E05U06DYAR, PigeonVision:TI_DYA0002A_SOD523_TPD1E05U06, F.Cu at (192.5, 127.6)
- added U13: TS3USB221DRCR, PigeonVision:TI_DRC0010J_VSON-10_3x3mm_P0.5mm, F.Cu at (182.5, 134.1)
- added U6: TPD4EUSB30DQAR, PigeonVision:TI_DQA0010A_USON-10_1x2.5mm_P0.5mm, F.Cu at (177.6, 58.4)
- added U7: LM61495RPHR, PigeonVision:TI_RPH0016_VQFN-HR-16_3.5x4.5mm, F.Cu at (122.8, 132.3)
- C1, C7: value 100nF -> 1uF; footprint PCM_JLCPCB:C_0402 -> PCM_JLCPCB:C_0805
- C10, C11, C12, C13, C18, C19, C20, C45, C47, C57: value 10uF -> 100nF; footprint Capacitor_SMD:C_1210_3225Metric -> PCM_JLCPCB:C_0402
- C2: value 220nF -> 100nF; footprint PCM_JLCPCB:C_0805 -> PCM_JLCPCB:C_0402
- C21: value 10uF -> 1uF; footprint Capacitor_SMD:C_1210_3225Metric -> PCM_JLCPCB:C_0805
- C22: value 10uF -> 33pF; footprint Capacitor_SMD:C_1210_3225Metric -> PCM_JLCPCB:C_0402
- C3: value 100nF -> 220nF; footprint PCM_JLCPCB:C_0402 -> PCM_JLCPCB:C_0805
- C30: value 33pF -> 10uF; footprint PCM_JLCPCB:C_0402 -> Capacitor_SMD:C_1210_3225Metric
- C33, C38, C43, C49, C50, C51, C61: value 100nF -> 10uF; footprint PCM_JLCPCB:C_0402 -> Capacitor_SMD:C_1210_3225Metric
- C5, C8: footprint PCM_JLCPCB:C_0603 -> PCM_JLCPCB:C_0805
- C9: value 220uF -> 100nF; footprint JLCImport_Auto:EEEFK1V221P -> PCM_JLCPCB:C_0402
- J1: value 10164227-1001A1RLF -> BATT CONN; footprint PigeonVision:Amphenol_10164227-1001A1RLF_2x50_P0.40mm -> Connector_AMASS:AMASS_XT60PW-M_1x02_P7.20mm_Horizontal
- J2: value 10164227-1001A1RLF -> PJ-102AH; footprint PigeonVision:Amphenol_10164227-1001A1RLF_2x50_P0.40mm_CM5_J2 -> PigeonVision:SameSky_PJ-102AH_Horizontal
- J3: value BATT CONN -> 10164227-1001A1RLF; footprint Connector_AMASS:AMASS_XT60PW-M_1x02_P7.20mm_Horizontal -> PigeonVision:Amphenol_10164227-1001A1RLF_2x50_P0.40mm
- J5: value PJ-102AH -> 10164227-1001A1RLF; footprint PigeonVision:SameSky_PJ-102AH_Horizontal -> PigeonVision:Amphenol_10164227-1001A1RLF_2x50_P0.40mm_CM5_J2
- R1: value 7.5kΩ -> 10kΩ
- R10: value 1kΩ -> 10
- R11, R22, R8: value 10kΩ -> 1kΩ
- R12: value 0Ω -> 2.2kΩ; footprint PCM_JLCPCB:R_0402 -> PCM_JLCPCB:R_0603
- R13: value 4.99kΩ -> 2.2kΩ
- R14: value 51kΩ -> 2.2kΩ; footprint PCM_JLCPCB:R_0402 -> PCM_JLCPCB:R_0603
- R2: value 1kΩ -> 7.5kΩ
- R21: value 1.5kΩ -> 39kΩ
- R23: value 0Ω -> 10kΩ
- R25: value 1kΩ -> 10kΩ
- R26: value 47kΩ -> 0Ω
- R28: value 0Ω -> 1.5kΩ; footprint PCM_JLCPCB:R_0603 -> PCM_JLCPCB:R_0402
- R29, R30: value 2.2kΩ -> 10kΩ; footprint PCM_JLCPCB:R_0603 -> PCM_JLCPCB:R_0402
- R3: value 51kΩ -> 1kΩ
- R4: value 4.7kΩ -> 56kΩ
- R5: value 10 -> 4.7kΩ
- R6: value 5mΩ -> 220Ω; footprint PigeonVision:Vishay_WSL2512_5mOhm_2W -> PCM_JLCPCB:R_0402
- R7: value 10 -> 5mΩ; footprint PCM_JLCPCB:R_0402 -> PigeonVision:Vishay_WSL2512_5mOhm_2W
- R9: value 39kΩ -> 10
- TP2: value 5V_MAIN -> 3V3_CAM
- TP3: value 5V_RF -> 5V_MAIN
- TP4: value 3V3_CAM -> GND
- TP7: value GND -> 5V_RF
- U1: value LM61495RPHR -> LM74502DDFR; footprint PigeonVision:TI_RPH0016_VQFN-HR-16_3.5x4.5mm -> PigeonVision:Texas_DDF0008A_SOT-8_1.6x2.9mm_P0.65mm
- U10: value BMP581 -> TPS62933FDRLR; footprint PigeonVision:Bosch_BMP581_LGA-10_2x2mm_P0.5mm -> PigeonVision:SOT-583-8
- U2: value LM74502DDFR -> INA226AIDGSR; footprint PigeonVision:Texas_DDF0008A_SOT-8_1.6x2.9mm_P0.65mm -> PigeonVision:TI_DGS0010A_VSSOP-10_3x3mm_P0.5mm
- U3: value INA226AIDGSR -> BMI088; footprint PigeonVision:TI_DGS0010A_VSSOP-10_3x3mm_P0.5mm -> PigeonVision:Bosch_LGA-16_4.5x3mm_P0.5mm_LayoutBorder7x1y_ClockwisePinNumbering
- U4: value TPS62933FDRLR -> BMP581; footprint PigeonVision:SOT-583-8 -> PigeonVision:Bosch_BMP581_LGA-10_2x2mm_P0.5mm
- U5: value 3.3uH -> TPD4EUSB30DQAR; footprint JLCImport_Auto:CYA1265-3_3UH -> PigeonVision:TI_DQA0010A_USON-10_1x2.5mm_P0.5mm
- U9: value BMI088 -> TPS62933FDRLR; footprint PigeonVision:Bosch_LGA-16_4.5x3mm_P0.5mm_LayoutBorder7x1y_ClockwisePinNumbering -> PigeonVision:SOT-583-8
- moved TP5 164.2 mm to (133.6, 116.3)
- moved TP6 164.2 mm to (133.6, 120.4)
- moved TP7 164.2 mm to (133.6, 124.4)
- moved J5 121.2 mm to (147.6, 68.4)
- moved C38 99.0 mm to (111.5, 137.7), turned to 0 degrees
- moved C32 96.0 mm to (105.9, 141.9), turned to 0 degrees
- moved R23 94.4 mm to (121.4, 128.2), turned to 0 degrees
- moved R22 91.8 mm to (121.4, 126.3), turned to 0 degrees
- moved C31 91.4 mm to (105.9, 137.7), turned to 0 degrees
- moved C39 91.4 mm to (111.5, 141.9), turned to 0 degrees
- moved TP4 89.9 mm to (129.6, 128.5), turned to 0 degrees
- moved R21 89.2 mm to (121.4, 124.5), turned to 0 degrees
- moved C33 89.0 mm to (111.5, 116.4), turned to 0 degrees
- moved C42 86.8 mm to (117.2, 124.9), turned to 0 degrees
- moved TP3 84.2 mm to (129.6, 124.4), turned to 0 degrees
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Connections:
- C1 pad 1: /Power & Regulators/VBAT_RAW -> 5V_MAIN
- C10 pad 1: VBAT -> GND
- C10 pad 2: GND -> 3V3_CM5
- C11 pad 1: VBAT -> Net-(U4-VDD)
- C12 pad 1: VBAT -> GND
- C12 pad 2: GND -> Net-(U4-CSB)
- C13 pad 1: VBAT -> GND
- C13 pad 2: GND -> /Ethernet/ETH_CT
- C14 pad 1: GND -> VBAT
- C14 pad 2: 5V_MAIN -> GND
- C15 pad 1: GND -> VBAT
- C15 pad 2: 5V_MAIN -> GND
- C16 pad 1: GND -> VBAT
- C16 pad 2: 5V_MAIN -> GND
- C17 pad 1: GND -> VBAT
- C17 pad 2: 5V_MAIN -> GND
- C18 pad 2: 5V_MAIN -> VBAT
- C19 pad 2: 5V_MAIN -> VBAT
- C2 pad 2: Net-(U2-VCAP) -> GND
- C20 pad 1: GND -> Net-(U7-CBOOT)
- C20 pad 2: 5V_MAIN -> Net-(U7-SW)
- C21 pad 1: GND -> /Power & Regulators/VBAT->5V_MAIN/VCC
- C21 pad 2: 5V_MAIN -> GND
- C22 pad 1: 5V_MAIN -> Net-(C22-Pad1)
- C22 pad 2: GND -> Net-(U7-FB)
- C23 pad 1: 5V_MAIN -> GND
- C23 pad 2: GND -> 5V_MAIN
- C25 pad 1: 5V_MAIN -> GND
- C25 pad 2: GND -> 5V_MAIN
- C27 pad 1: 5V_MAIN -> GND
- C27 pad 2: GND -> 5V_MAIN
- C29 pad 1: 5V_MAIN -> GND
- C29 pad 2: GND -> 5V_MAIN
- C3 pad 1: 3V3_CM5 -> /Power & Regulators/VBAT_RAW
- C3 pad 2: GND -> Net-(U1-VCAP)
- C30 pad 1: Net-(C30-Pad1) -> 5V_MAIN
- C30 pad 2: Net-(U1-FB) -> GND
- C31 pad 1: VBAT -> GND
- C31 pad 2: GND -> 5V_MAIN
- C32 pad 1: VBAT -> 5V_MAIN
- C33 pad 2: VBAT -> 5V_MAIN
- C38 pad 1: Net-(U4-SW) -> 5V_MAIN
- C38 pad 2: Net-(C38-Pad2) -> GND
- C39 pad 1: 5V_RF -> GND
- C39 pad 2: GND -> Net-(C39-Pad2)
- C40 pad 1: 5V_RF -> Net-(C39-Pad2)
- C41 pad 1: 5V_RF -> GND
- C41 pad 2: GND -> Net-(C41-Pad2)
- C42 pad 1: 5V_RF -> Net-(C41-Pad2)
- C43 pad 1: GND -> VBAT
- C43 pad 2: Net-(U4-SS) -> GND
- C44 pad 1: 5V_RF -> VBAT
- C45 pad 1: 5V_RF -> GND
- C45 pad 2: GND -> VBAT
- C46 pad 2: 5V_RF -> Net-(U9-SS)
- C47 pad 1: VBAT -> Net-(U9-SW)
- C47 pad 2: GND -> Net-(C47-Pad2)
- C48 pad 2: VBAT -> 5V_RF
- C49 pad 1: GND -> 5V_RF
- C49 pad 2: Net-(U8-SS) -> GND
- C5 pad 1: /Power & Regulators/VBAT->5V_MAIN/VCC -> Net-(U2-Vin+)
- C5 pad 2: GND -> Net-(U2-Vin-)
- C50 pad 1: Net-(U8-SW) -> 5V_RF
- C50 pad 2: Net-(C50-Pad2) -> GND
- C51 pad 1: GND -> 5V_RF
- C51 pad 2: 3V3_CAM -> GND
- C52 pad 1: 3V3_CAM -> 5V_RF
- C53 pad 1: 3V3_CAM -> 5V_RF
- C54 pad 1: 3V3_CAM -> 5V_RF
- C55 pad 1: 3V3_CAM -> VBAT
- C56 pad 1: 3V3_CAM -> VBAT
- C57 pad 1: 3V3_CAM -> GND
- C57 pad 2: GND -> VBAT
- C58 pad 1: Net-(U10-VDD) -> GND
- C58 pad 2: GND -> Net-(U10-SS)
- C59 pad 1: GND -> Net-(U10-SW)
- C59 pad 2: Net-(U10-CSB) -> Net-(C59-Pad2)
- C6 pad 1: GND -> 3V3_CM5
- C6 pad 2: VBAT -> GND
- C60 pad 2: 3V3_CM5 -> 3V3_CAM
- C61 pad 1: 3V3_CM5 -> 3V3_CAM
- C7 pad 1: GND -> 3V3_CAM
- C7 pad 2: VBAT -> GND
- C8 pad 1: Net-(U3-Vin+) -> 3V3_CAM
- C8 pad 2: Net-(U3-Vin-) -> GND
- C9 pad 1: VBAT -> 3V3_CM5
- J1 pad 2: GND -> /Power & Regulators/VBAT_RAW
- J2 pad 1: unconnected-(J2-USB_OTG_ID-Pad1) -> /Power & Regulators/VBAT_RAW
- J2 pad 2: unconnected-(J2-PCIe_nCLKREQ-Pad2) -> GND
- J2 pad 3: unconnected-(J2-USB2_N-Pad3) -> GND
- J3 pad 2: /Power & Regulators/VBAT_RAW -> GND
- J5 pad 1: /Power & Regulators/VBAT_RAW -> unconnected-(J5-USB_OTG_ID-Pad1)
- J5 pad 2: GND -> unconnected-(J5-PCIe_nCLKREQ-Pad2)
- J5 pad 3: GND -> /CM5/USB2_N
- Q1 pad 1: Net-(U2-SRC) -> Net-(U1-SRC)
- Q1 pad 2: Net-(U2-SRC) -> Net-(U1-SRC)
- Q1 pad 3: Net-(U2-SRC) -> Net-(U1-SRC)
- Q2 pad 1: Net-(U2-SRC) -> Net-(U1-SRC)
- Q2 pad 2: Net-(U2-SRC) -> Net-(U1-SRC)
- Q2 pad 3: Net-(U2-SRC) -> Net-(U1-SRC)
- R1 pad 1: /Power & Regulators/VBAT_RAW -> /CM5/FAN_PWM
- R1 pad 2: /Power & Regulators/PWR_EN -> 3V3_CM5
- R10 pad 1: Net-(R10-Pad1) -> VBAT
- R10 pad 2: Net-(U1-FB) -> Net-(U2-Vin-)
- R11 pad 1: GND -> 5V_RF
- R11 pad 2: /CM5/5V_RF_EN -> Net-(LED3-A)
- R12 pad 1: Net-(U1-RBOOT) -> 3V3_CM5
- R12 pad 2: Net-(U1-CBOOT) -> /CM5/CAM1_I2C_SCL
- R13 pad 1: 5V_MAIN -> 3V3_CM5
- R13 pad 2: Net-(C30-Pad1) -> /CM5/CAM1_I2C_SDA
- R14 pad 1: 5V_RF -> 3V3_CM5
- R14 pad 2: Net-(R14-Pad2) -> /CM5/CAM1_RST
- R2 pad 1: /Power & Regulators/PWR_EN -> /Power & Regulators/VBAT_RAW
- R2 pad 2: GND -> /Power & Regulators/PWR_EN
- R21 pad 1: Net-(R14-Pad2) -> 5V_MAIN
- R21 pad 2: Net-(U4-FB) -> Net-(R21-Pad2)
- R22 pad 1: Net-(U4-FB) -> Net-(R21-Pad2)
- R22 pad 2: GND -> Net-(U7-FB)
- R23 pad 1: Net-(U4-BST) -> Net-(U7-FB)
- R23 pad 2: Net-(C38-Pad2) -> GND
- R25 pad 1: 5V_RF -> GND
- R25 pad 2: Net-(LED2-A) -> /CM5/5V_RF_EN
- R26 pad 1: 3V3_CAM -> Net-(U9-BST)
- R26 pad 2: Net-(U8-FB) -> Net-(C47-Pad2)
- R28 pad 1: Net-(U10-INT) -> Net-(R27-Pad2)
- R28 pad 2: GND -> Net-(U9-FB)
- R29 pad 1: 3V3_CM5 -> Net-(U9-FB)
- R29 pad 2: /CM5/CAM1_I2C_SDA -> GND
- R3 pad 1: /Power & Regulators/VBAT_RAW -> /Power & Regulators/PWR_EN
- R3 pad 2: Net-(U2-OV) -> GND
- R30 pad 1: 3V3_CM5 -> GND
- R30 pad 2: /Cameras/CAM1_RST -> 3V3_CM5
- R4 pad 1: Net-(U2-OV) -> /Power & Regulators/VBAT_RAW
- R4 pad 2: GND -> Net-(U1-OV)
- R5 pad 1: Net-(Q2-D) -> Net-(U1-OV)
- R5 pad 2: Net-(U3-Vin+) -> GND
- R6 pad 1: Net-(Q2-D) -> 3V3_CAM
- R6 pad 2: VBAT -> Net-(LED1-A)
- R7 pad 1: VBAT -> Net-(Q2-D)
- R7 pad 2: Net-(U3-Vin-) -> VBAT
- R8 pad 1: Net-(U1-FB) -> 5V_MAIN
- R8 pad 2: GND -> Net-(LED2-A)
- R9 pad 1: 5V_MAIN -> Net-(Q2-D)
- R9 pad 2: Net-(R10-Pad1) -> Net-(U2-Vin+)
- TP2 pad 1: 5V_MAIN -> 3V3_CAM
- TP3 pad 1: 5V_RF -> 5V_MAIN
- TP4 pad 1: 3V3_CAM -> GND
- TP7 pad 1: GND -> 5V_RF
- U1 pad 1: GND -> /Power & Regulators/PWR_EN
- U1 pad 2: VBAT -> GND
- U1 pad 3: Net-(U1-RBOOT) -> unconnected-(U1-NC-Pad3)
- U1 pad 4: Net-(U1-CBOOT) -> Net-(U1-VCAP)
- U1 pad 5: 5V_MAIN -> /Power & Regulators/VBAT_RAW
- U1 pad 6: /Power & Regulators/VBAT->5V_MAIN/VCC -> Net-(Q1-G)
- U1 pad 7: Net-(U1-FB) -> Net-(U1-OV)
- U1 pad 8: GND -> Net-(U1-SRC)
- U10 pad 1: Net-(U10-CSB) -> unconnected-(U10-RT-Pad1)
- U10 pad 2: /Sensors/SENSOR_I2C_SCL -> 3V3_CM5
- U10 pad 3: GND -> VBAT
- U10 pad 4: /Sensors/SENSOR_I2C_SDA -> GND
- U10 pad 5: GND -> Net-(U10-SW)
- U10 pad 6: Net-(U10-CSB) -> Net-(U10-BST)
- U10 pad 7: Net-(U10-INT) -> Net-(U10-SS)
- U10 pad 8: GND -> Net-(U10-FB)
- U2 pad 1: /Power & Regulators/PWR_EN -> GND
- U2 pad 4: Net-(U2-VCAP) -> /Sensors/SENSOR_I2C_SDA
- U2 pad 5: /Power & Regulators/VBAT_RAW -> /Sensors/SENSOR_I2C_SCL
- U2 pad 6: Net-(Q1-G) -> 3V3_CM5
- U2 pad 7: Net-(U2-OV) -> GND
- U2 pad 8: Net-(U2-SRC) -> Net-(Q2-D)
- U3 pad 1: GND -> unconnected-(U3-INT2-Pad1)
- U3 pad 10: Net-(U3-Vin+) -> GND
- U3 pad 3: unconnected-(U3-~{Alert}-Pad3) -> 3V3_CM5
- U3 pad 4: /Sensors/SENSOR_I2C_SDA -> GND
- U3 pad 5: /Sensors/SENSOR_I2C_SCL -> unconnected-(U3-~{CSB2}-Pad5)
- U3 pad 6: 3V3_CM5 -> GND
- U3 pad 7: GND -> 3V3_CM5
- U3 pad 8: Net-(Q2-D) -> /Sensors/SENSOR_I2C_SCL
- U3 pad 9: Net-(U3-Vin-) -> /Sensors/SENSOR_I2C_SDA
- U4 pad 1: unconnected-(U4-RT-Pad1) -> Net-(U4-CSB)
- U4 pad 2: /CM5/5V_RF_EN -> /Sensors/SENSOR_I2C_SCL
- U4 pad 3: VBAT -> GND
- U4 pad 4: GND -> /Sensors/SENSOR_I2C_SDA
- U4 pad 5: Net-(U4-SW) -> GND
- U4 pad 6: Net-(U4-BST) -> Net-(U4-CSB)
- U4 pad 7: Net-(U4-SS) -> Net-(U4-INT)
- U4 pad 8: Net-(U4-FB) -> GND
- U5 pad 1: Net-(U1-SW) -> /CM5/ETH0_P
- U5 pad 2: 5V_MAIN -> /CM5/ETH0_N
- U9 pad 2: GND -> /CM5/5V_RF_EN
- U9 pad 3: 3V3_CM5 -> VBAT
- U9 pad 5: unconnected-(U9-~{CSB2}-Pad5) -> Net-(U9-SW)
- U9 pad 6: GND -> Net-(U9-BST)
- U9 pad 7: 3V3_CM5 -> Net-(U9-SS)
- U9 pad 8: /Sensors/SENSOR_I2C_SCL -> Net-(U9-FB)
Other:
- board outline removed
- rule solder_mask_min_width: 0.10 -> 0.1
