File: hardware/carrier/PigeonCarrier/PigeonCarrier.kicad_pcb (KiCad board)
At the start: 4 copper layers, 139 parts, among them J1 BATT CONN, J10 USB4105_GF_A, J11 Samtec_TSM-102-01-L-SV-P-TR, J2 PJ-102AH, J3 10164227-1001A1RLF, J4 BM04B-SRSS-TB(LF)(SN), J5 10164227-1001A1RLF, J7 FH12-22S-0.5SH(55), J8 FH12-22S-0.5SH(55), J9 A70-112-331N126, Q1 CSD18540Q5B, Q2 CSD18540Q5B, Q3 BSS138BK,215, SW1 PTS636 SK25 SMTR LFS, U1 LM74502DDFR, U10 TPS62933FDRLR, U11 TPD4E05U06DQAR, U12 TPD1E05U06DYAR, U13 TS3USB221DRCR, U2 INA226AIDGSR, U3 BMI088, U4 BMP581, U5 TPD4EUSB30DQAR, U6 TPD4EUSB30DQAR, U7 LM61495RPHR, U9 TPS62933FDRLR

Commit message: finished rough layout
Parts:
- added C4: 220uF, PigeonVision:Panasonic_EEE-FK1V221P_CaseF_8x10.2mm, F.Cu at (62.3, 79.7)
- added H1: MountingHole_3-8in_Rod_NPTH_10.32mm, MountingHole_3-8in_Rod_NPTH_10.32mm, F.Cu at (30.0, 100.0)
- added H2: MountingHole_3-8in_Rod_NPTH_10.32mm, MountingHole_3-8in_Rod_NPTH_10.32mm, F.Cu at (150.0, 100.0)
- added J12: UART, PigeonVision:JST_SH_BM03B-SRSS-TB_1x03-1MP_P1.00mm_Vertical, F.Cu at (147.2, 64.7)
- added J6: PULL_PIN, Connector_AMASS:AMASS_XT30PW-M_1x02_P2.50mm_Horizontal, F.Cu at (37.3, 85.1)
- added L1: 6.8uH, JLCImport_Auto:CYA1040-6_8UH, F.Cu at (53.5, 115.7)
- added L2: 6.8uH, JLCImport_Auto:CYA1040-6_8UH, F.Cu at (53.5, 132.9)
- added L3: 3.3uH, JLCImport_Auto:CYA1265-3_3UH, F.Cu at (50.0, 95.2)
- added LED1: 0805G_Green, JLCImport_Auto:0805G_Green, F.Cu at (55.8, 123.9)
- added LED2: 0805G_Green, JLCImport_Auto:0805G_Green, F.Cu at (69.0, 86.8)
- added LED3: 0805G_Green, JLCImport_Auto:0805G_Green, F.Cu at (55.8, 106.7)
- added LED4: 0805G_Green, JLCImport_Auto:0805G_Green, F.Cu at (129.4, 75.1)
- added R39: 1kΩ, PCM_JLCPCB:R_0402, F.Cu at (134.1, 69.9)
- added R40: 1kΩ, PCM_JLCPCB:R_0402, F.Cu at (133.6, 68.7)
- added R41: 220Ω, PCM_JLCPCB:R_0402, F.Cu at (129.5, 73.1)
- added REF**: ANTSDR E200 - planning, PigeonVision:MicroPhase_ANTSDR_E200_Mounting_80x50mm_Planning, F.Cu at (100.4, 129.5)
- Q1, Q2: footprint Package_TO_SOT_SMD:TDSON-8-1 -> PigeonVision:TI_CSD18540Q5B_Q5B
- R10, R9: value 10 -> 10Ω
- R15, R16: value 10 -> 10Ω; footprint PigeonVision:KiCad_Resistor_SMD_R_0402_1005Metric -> PCM_JLCPCB:R_0402
- moved C45 156.1 mm to (47.0, 110.0), turned to 90 degrees
- moved R25 153.2 mm to (47.0, 108.0), turned to -90 degrees
- moved C57 152.8 mm to (47.0, 127.2), turned to 90 degrees
- moved C46 152.6 mm to (49.0, 107.0)
- moved R30 150.3 mm to (47.0, 125.2), turned to -90 degrees
- moved C47 150.3 mm to (51.5, 109.0)
- moved C58 149.5 mm to (49.0, 124.2)
- moved C43 149.3 mm to (44.5, 111.7), turned to -90 degrees
- moved U9 149.2 mm to (49.1, 109.0)
- moved R26 148.3 mm to (51.5, 107.7)
- moved U10 147.2 mm to (49.1, 126.2)
- moved C59 147.1 mm to (51.5, 126.2)
- moved C44 146.4 mm to (44.5, 107.0), turned to 90 degrees
- moved C55 145.9 mm to (44.5, 128.9), turned to -90 degrees
- moved R31 145.4 mm to (51.5, 124.9)
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Connections:
- net /CM5/ETH_LED_K renamed /CM5/ETH_LED_Y
- C39 pad 2: Net-(C39-Pad2) -> 5V_MAIN
- C40 pad 1: Net-(C39-Pad2) -> 5V_MAIN
- C41 pad 2: Net-(C41-Pad2) -> 5V_MAIN
- C42 pad 1: Net-(C41-Pad2) -> 5V_MAIN
- J3 pad 21: unconnected-(J3-LED_nACT-Pad21) -> /CM5/LED_nACT
- J3 pad 51: unconnected-(J3-GPIO15-Pad51) -> /CM5/UART_RX
- J3 pad 55: unconnected-(J3-GPIO14-Pad55) -> /CM5/UART_TX
- MP1 pad 1: (no net) -> GND
- MP1 pad 2: (no net) -> GND
- MP1 pad 3: (no net) -> GND
- MP1 pad 4: (no net) -> GND
Other:
- board outline added: 144.8 x 144.8 mm
