File: hardware/carrier/PigeonCarrier/PigeonCarrier.kicad_pcb (KiCad board)
At the start: 4 copper layers, 144.8 x 144.8 mm, 155 parts, among them J1 BATT CONN, J10 USB4105_GF_A, J11 Samtec_TSM-102-01-L-SV-P-TR, J12 UART, J2 PJ-102AH, J3 10164227-1001A1RLF, J4 BM04B-SRSS-TB(LF)(SN), J5 10164227-1001A1RLF, J6 PULL_PIN, J7 FH12-22S-0.5SH(55), J8 FH12-22S-0.5SH(55), J9 A70-112-331N126, Q1 CSD18540Q5B, Q2 CSD18540Q5B, Q3 BSS138BK,215, SW1 PTS636 SK25 SMTR LFS, U1 LM74502DDFR, U10 TPS62933FDRLR, U11 TPD4E05U06DQAR, U12 TPD1E05U06DYAR, U13 TS3USB221DRCR, U2 INA226AIDGSR, U3 BMI088, U4 BMP581, U5 TPD4EUSB30DQAR, U6 TPD4EUSB30DQAR, U7 LM61495RPHR, U9 TPS62933FDRLR

Commit message: Update carrier placement and vertical connector libraries
Save the latest component placements and mechanical mounting changes. Include the vertical XT60/XT30 and camera connector symbols, footprints, redistributable CAD, licenses and documentation. Keep local-only vendor models ignored.

Validation: ERC has zero findings. Native KiCad loading and netlist comparison confirm all 152 schematic components and 681 numbered pads agree. Full DRC could not complete because the KiCad CLI aborted in this environment.
Parts:
- J1: footprint Connector_AMASS:AMASS_XT60PW-M_1x02_P7.20mm_Horizontal -> PigeonVision:AMASS_XT60PB-M_1x02_P7.20mm_Vertical_2025
- J6: footprint Connector_AMASS:AMASS_XT30PW-M_1x02_P2.50mm_Horizontal -> PigeonVision:AMASS_XT30UPB-M_1x02_P5.00mm_Vertical_2025
- J7, J8: value FH12-22S-0.5SH(55) -> FH12-22S-0.5SVA(54); footprint PigeonVision:Hirose_FH12-22S-0.5SH_1x22-1MP_P0.50mm_Horizontal -> PigeonVision:Hirose_FH12-22S-0.5SVA_1x22_P0.50mm_Vertical
- moved C55 47.1 mm to (73.4, 91.7), turned to 180 degrees
- moved C56 46.7 mm to (78.2, 91.7), turned to 0 degrees
- moved C57 43.3 mm to (75.2, 94.2), turned to 0 degrees
- moved R30 43.2 mm to (77.2, 94.2), turned to 180 degrees
- moved J6 41.6 mm to (54.1, 47.0), turned to -75 degrees
- moved U10 40.4 mm to (76.2, 96.2), turned to -90 degrees
- moved C58 40.3 mm to (78.2, 96.2), turned to -90 degrees
- moved C59 36.9 mm to (76.2, 98.7), turned to -90 degrees
- moved R31 36.8 mm to (77.4, 98.7), turned to -90 degrees
- moved L2 35.9 mm to (69.4, 100.7), turned to -90 degrees
- moved R33 33.7 mm to (76.2, 101.0), turned to 90 degrees
- moved LED1 33.6 mm to (79.8, 100.5), turned to -90 degrees
- moved R6 29.7 mm to (79.8, 103.2), turned to 0 degrees
- moved TP4 29.3 mm to (44.8, 121.5), turned to -90 degrees
- moved C60 29.3 mm to (65.9, 107.7), turned to 0 degrees
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