File: hardware/carrier/PigeonCarrier/Ethernet.kicad_sch (KiCad schematic)
At the start: 0 parts

Commit message: Update carrier schematics, parts library, and JLC rules
Parts:
- added C13: 100nF, PCM_JLCPCB:C_0402, symbol PCM_JLCPCB-Capacitors:0402,100nF,(2)
- added J9: A70-112-331N126, PigeonVision:RJ45_EDAC_A70-112-331N126, symbol PigeonVision:A70-112-331N126
- added R18, R19: 470Ω, PCM_JLCPCB:R_0402, symbol PCM_JLCPCB-Resistors:0402,470Ω
- added U5, U6: TPD4EUSB30DQAR, PigeonVision:TI_DQA0010A_USON-10_1x2.5mm_P0.5mm, symbol PigeonVision:TPD4EUSB30DQAR
Connections:
- new net: J9.16 (LEDG_K), R18.1
- new net: J9.18 (LEDY_K), R19.1
- new net 3V3_CM5: J9.15 (LEDG_A), J9.17 (LEDY_A)
- new net ETH0_N: J9.2 (TRD0-), U5.2 (D1-), U5.9 (NC)
- new net ETH0_P: J9.1 (TRD0+), U5.1 (D1+), U5.10 (NC)
- new net ETH1_N: J9.6 (TRD1-), U5.5 (D2-), U5.6 (NC)
- new net ETH1_P: J9.3 (TRD1+), U5.4 (D2+), U5.7 (NC)
- new net ETH2_N: J9.8 (TRD2-), U6.2 (D1-), U6.9 (NC)
- new net ETH2_P: J9.7 (TRD2+), U6.1 (D1+), U6.10 (NC)
- new net ETH3_N: J9.10 (TRD3-), U6.5 (D2-), U6.6 (NC)
- new net ETH3_P: J9.9 (TRD3+), U6.4 (D2+), U6.7 (NC)
- new net ETH_CT: C13.2, J9.4 (CT), J9.5 (CT)
- new net ETH_LED_G: R18.2
- new net ETH_LED_K: R19.2
- new net GND: C13.1, J9.19 (SHIELD), J9.20 (SHIELD), U5.3 (GND), U5.8 (GND), U6.3 (GND), U6.8 (GND)
- no-connect marks 0 -> 4
Other:
- note added: "Gigabit Ethernet"
- note added: "Magnetics + RJ45"
- note added: "TVS"

Commit message: update updategit statusgit status
Changed lines of the file:
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@@
 	)
 	(label "ETH1_N"
-		(at 83.82 91.44 0)
+		(at 82.55 91.44 0)
 		(effects
 			(font
@@
 		)
 	)
+	(netclass_flag ""
+		(length 2.54)
+		(shape dot)
+		(at 94.0085 110.49 0)
+		(effects
+			(font
+				(size 1.27 1.27)
+			)
+			(justify left bottom)
+		)
+		(property "Net Class" "ETH_100R"
+			(at 92.9925 107.442 0)
+			(show_name no)
+			(do_not_autoplace no)
+			(effects
+				(font
+					(size 0.9 0.9)
+					(italic yes)
+				)
+				(justify right)
+			)
+		)
+	)
+	(netclass_flag ""
+		(length 2.54)
+		(shape dot)
+		(at 95.25 88.9 0)
+		(effects
+			(font
+				(size 1.27 1.27)
+			)
+			(justify left bottom)
+		)
+		(property "Net Class" "ETH_100R"
+			(at 94.234 85.852 0)
+			(show_name no)
+			(do_not_autoplace no)
+			(effects
+				(font
+					(size 0.9 0.9)
+					(italic yes)
+				)
+				(justify right)
+			)
+		)
+	)
+	(netclass_flag ""
+		(length 2.54)
+		(shape dot)
+		(at 158.75 81.28 0)
+		(effects
+			(font
+				(size 1.27 1.27)
+			)
+			(justify left bottom)
+		)
+		(property "Net Class" "ETH_100R"
+			(at 157.734 78.232 0)
+			(show_name no)
+			(do_not_autoplace no)
+			(effects
+				(font
+					(size 0.9 0.9)
+					(italic yes)
+				)
+				(justify right)
+			)
+		)
+	)
+	(netclass_flag ""
+		(length 2.54)
+		(shape dot)
+		(at 95.25 81.28 0)
+		(effects
+			(font
+				(size 1.27 1.27)
+			)
+			(justify left bottom)
+		)
+		(property "Net Class" "ETH_100R"
+			(at 94.234 78.232 0)
+			(show_name no)
+			(do_not_autoplace no)
+			(effects
+				(font
+					(size 0.9 0.9)
+					(italic yes)
+				)
+				(justify right)
+			)
+		)
+	)
+	(netclass_flag ""
+		(length 2.54)
+		(shape dot)
+		(at 158.7105 104.14 0)
+		(effects
+			(font
+				(size 1.27 1.27)
+			)
+			(justify left bottom)
+		)
+		(property "Net Class" "ETH_100R"
+			(at 157.6945 101.092 0)
+			(show_name no)
+			(do_not_autoplace no)
+			(effects
+				(font
+					(size 0.9 0.9)
+					(italic yes)
+				)
+				(justify right)
+			)
+		)
+	)
+	(netclass_flag ""
+		(length 2.54)
+		(shape dot)
+		(at 93.98 118.11 0)
+		(effects
+			(font
+				(size 1.27 1.27)
+			)
+			(justify left bottom)
+		)
+		(property "Net Class" "ETH_100R"
+			(at 92.964 115.062 0)
+			(show_name no)
+			(do_not_autoplace no)
+			(effects
+				(font
+					(size 0.9 0.9)
+					(italic yes)
+				)
+				(justify right)
+			)
+		)
+	)
+	(netclass_flag ""
+		(length 2.54)
+		(shape dot)
+		(at 158.75 88.9 0)
+		(effects
+			(font
+				(size 1.27 1.27)
+			)
+			(justify left bottom)
+		)
+		(property "Net Class" "ETH_100R"
+			(at 157.734 85.852 0)
+			(show_name no)
+			(do_not_autoplace no)
+			(effects
+				(font
+					(size 0.9 0.9)
+					(italic yes)
+				)
+				(justify right)
+			)
+		)
+	)
+	(netclass_flag ""
+		(length 2.54)
+		(shape dot)
+		(at 158.7105 96.52 0)
+		(effects
+			(font
+				(size 1.27 1.27)
+			)
+			(justify left bottom)
+		)
+		(property "Net Class" "ETH_100R"
+			(at 157.6945 93.472 0)
+			(show_name no)
+			(do_not_autoplace no)
+			(effects
+				(font
+					(size 0.9 0.9)
+					(italic yes)
+				)
+				(justify right)
+			)
+		)
+	)

Commit message: finished rough layout
Parts:
- C13: MPN (none) -> CL05B104KB54PNC
- R18, R19: MPN (none) -> 0402WGF4700TCE
Connections:
- net ETH_LED_K renamed ETH_LED_Y
Changed lines of the file:
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@@
 		)
 	)
-	(hierarchical_label "ETH_LED_K"
+	(hierarchical_label "ETH_LED_Y"
 		(shape input)
 		(at 219.71 104.14 0)
@@
 			)
 		)
+		(property "MPN" "0402WGF4700TCE"
+			(at 214.63 104.14 0)
+			(hide yes)
+			(show_name no)
+			(do_not_autoplace no)
+			(effects
+				(font
+					(size 1.27 1.27)
+				)
+			)
+		)
 		(pin "1"
 		)
@@
 			)
 		)
+		(property "MPN" "CL05B104KB54PNC"
+			(at 165.1 118.11 0)
+			(hide yes)
+			(show_name no)
+			(do_not_autoplace no)
+			(effects
+				(font
+					(size 1.27 1.27)
+				)
+			)
+		)
 		(pin "1"
 		)
@@
 			(at 214.63 96.52 0)
 			(hide yes)
+			(show_name no)
+			(do_not_autoplace no)
+			(effects
+				(font
+					(size 1.27 1.27)
+				)
+			)
+		)
+		(property "MPN" "0402WGF4700TCE"
+			(at 214.63 96.52 0)
+			(hide yes)
