File: hardware/carrier/PigeonCarrier/Sensors.kicad_sch (KiCad schematic)
At the start: 0 parts

Commit message: Update carrier schematics, parts library, and JLC rules
Parts:
- added C10, C11, C12, C9: 100nF, PCM_JLCPCB:C_0402, symbol PCM_JLCPCB-Capacitors:0402,100nF,(2)
- added R15, R16: 10, PigeonVision:KiCad_Resistor_SMD_R_0402_1005Metric, symbol Device:R
- added R17: 0Ω, PCM_JLCPCB:R_0603, symbol PCM_JLCPCB-Resistors:0603,0Ω
- added U3: BMI088, PigeonVision:Bosch_LGA-16_4.5x3mm_P0.5mm_LayoutBorder7x1y_ClockwisePinNumbering, symbol PigeonVision:BMI088
- added U4: BMP581, PigeonVision:Bosch_BMP581_LGA-10_2x2mm_P0.5mm, symbol PigeonVision:BMP581
Connections:
- new net: C12.2, R16.2, U4.1 (VDDIO), U4.6 (CSB)
- new net: C11.1, R15.2, U4.10 (VDD)
- new net: R17.1, U4.7 (INT)
- new net 3V3_CM5: C10.2, C9.1, R15.1, R16.1, U3.11 (VDDIO), U3.14 (~{CSB1}), U3.3 (VDD), U3.7 (PS)
- new net GND: C10.1, C11.2, C12.1, C9.2, R17.2, U3.10 (SDO2), U3.15 (SDO1), U3.2 (GNDA), U3.4 (GNDA), U3.6 (GNDIO), U4.3 (VSS), U4.5 (SDO/ADDR), U4.8 (VSS), U4.9 (VSS)
- new net SENSOR_I2C_SCL: U3.8 (SCK/SCL), U4.2 (SCK/SCL)
- new net SENSOR_I2C_SDA: U3.9 (SDI/SDA), U4.4 (SDI/SDA)
- no-connect marks 0 -> 5
Other:
- note added: "BMI088 inertial sensor"
- note added: "BMP581 pressure sensor"
- note added: "Settings / calculations: Design Master, Power budget A91:F103"

Commit message: finished rough layout
Parts:
- C10, C11, C12, C9: MPN (none) -> CL05B104KB54PNC
- R15, R16: value 10 -> 10Ω; footprint PigeonVision:KiCad_Resistor_SMD_R_0402_1005Metric -> PCM_JLCPCB:R_0402; symbol Device:R -> PCM_JLCPCB-Resistors:0402,10Ω; Attrition Qty (none) -> 10; Category (none) -> Resistors,Chip Resistor - Surface Mount; Class (none) -> Basic Component; DigiKey Part # 311-10.0LRCT-ND -> (none); LCSC (none) -> C25077; LCSC Part # C138066 -> C25077; MPN RC0402FR-0710RL -> 0402WGF100JTCE; Manufacturer YAGEO -> UNI-ROYAL(Uniroyal Elec); Minimum Qty (none) -> 20; Operating Temperature Range (none) -> -55°C~+155°C; Overload Voltage (Max) (none) -> 50V; Part (none) -> 0402WGF100JTCE; Power(Watts) (none) -> 62.5mW; Price (none) -> 0.004USD; Process (none) -> SMT; Resistance (none) -> 10Ω; Stock (none) -> 4873481; Temperature Coefficient (none) -> ±200ppm/°C; Tolerance 1% -> ±1%; Type (none) -> Thick Film Resistors
- R17: MPN (none) -> 0603WAF0000T5E
Other:
- note removed: "Settings / calculations: Design Master, Power budget A91:F103"
- moved on the sheet: C10, C9, U3
