File: hardware/carrier/PigeonCarrier/Service_USB.kicad_sch (KiCad schematic)
At the start: 13 parts, among them J10 USB4105_GF_A, J11 Samtec_TSM-102-01-L-SV-P-TR, Q3 BSS138BK,215, SW1 PTS636 SK25 SMTR LFS, U11 TPD4E05U06DQAR, U12 TPD1E05U06DYAR, U13 TS3USB221DRCR

Commit message: finished rough layout
Parts:
- C67: MPN (none) -> CL05B104KB54PNC
- R34, R35: MPN (none) -> 0402WGF5101TCE
- R36: MPN (none) -> 0402WGF1001TCE
- R37, R38: MPN (none) -> 0402WGF1002TCE
Changed lines of the file:
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@@
 	(text "Data Switch"
 		(exclude_from_sim no)
-		(at 213.36 35.56 0)
+		(at 206.756 52.324 0)
 		(effects
 			(font
@@
 		)
 	)
+	(netclass_flag ""
+		(length 2.54)
+		(shape dot)
+		(at 250.19 66.04 0)
+		(effects
+			(font
+				(size 1.27 1.27)
+			)
+			(justify left bottom)
+		)
+		(property "Net Class" "USB_90R"
+			(at 249.174 62.992 0)
+			(show_name no)
+			(do_not_autoplace no)
+			(effects
+				(font
+					(size 0.9 0.9)
+					(italic yes)
+				)
+				(justify right)
+			)
+		)
+	)
+	(netclass_flag ""
+		(length 2.54)
+		(shape dot)
+		(at 60.96 63.5 0)
+		(effects
+			(font
+				(size 1.27 1.27)
+			)
+			(justify left bottom)
+		)
+		(property "Net Class" "USB_90R"
+			(at 59.944 60.452 0)
+			(show_name no)
+			(do_not_autoplace no)
+			(effects
+				(font
+					(size 0.9 0.9)
+					(italic yes)
+				)
+				(justify right)
+			)
+		)
+	)
 	(symbol
 		(lib_id "PCM_JLCPCB-Resistors:0402,10kΩ")
@@
 			)
 		)
+		(property "MPN" "0402WGF1002TCE"
+			(at 177.8 57.15 0)
+			(hide yes)
+			(show_name no)
+			(do_not_autoplace no)
+			(effects
+				(font
+					(size 1.27 1.27)
+				)
+			)
+		)
 		(pin "1"
 		)
@@
 			)
 		)
+		(property "MPN" "0402WGF1002TCE"
+			(at 167.64 73.66 0)
+			(hide yes)
+			(show_name no)
+			(do_not_autoplace no)
+			(effects
+				(font
+					(size 1.27 1.27)
+				)
+			)
+		)
 		(pin "1"
 		)
@@
 			)
 		)
+		(property "MPN" "0402WGF5101TCE"
+			(at 63.5 55.88 0)
+			(hide yes)
+			(show_name no)
+			(do_not_autoplace no)
+			(effects
+				(font
+					(size 1.27 1.27)
+				)
+			)
+		)
 		(pin "1"
 		)
@@
 			)
 		)
+		(property "MPN" "0402WGF1001TCE"
+			(at 161.29 68.58 0)
+			(hide yes)
+			(show_name no)
+			(do_not_autoplace no)
+			(effects
+				(font
+					(size 1.27 1.27)
+				)
+			)
+		)
 		(pin "1"
 		)
@@
 			)
 		)
+		(property "MPN" "CL05B104KB54PNC"
+			(at 238.76 58.42 0)
+			(hide yes)
+			(show_name no)
+			(do_not_autoplace no)
+			(effects
+				(font
+					(size 1.27 1.27)
+				)
+			)
+		)
 		(pin "1"
 		)
@@
 			(at 63.5 58.42 0)
 			(hide yes)
+			(show_name no)
+			(do_not_autoplace no)
+			(effects
+				(font
+					(size 1.27 1.27)
+				)
+			)
+		)
+		(property "MPN" "0402WGF5101TCE"
+			(at 63.5 58.42 0)
+			(hide yes)
