File: hardware/carrier/PigeonCarrier/batt_5V_sdr.kicad_sch (KiCad schematic)
At the start: 19 parts, among them U4 TPS62933FDRLR

Commit message: Update carrier schematics, parts library, and JLC rules
Parts:
- renumbered C32 to C43, C31 to C44, C33 to C45, C43 to C46, C38 to C47, C46 to C48, C39 to C49, C40 to C50, C41 to C51, C42 to C52, C44 to C53, C45 to C54, R11 to R25, R23 to R26, R14 to R27, R21 to R28, R22 to R29, U4 to U9
Other:
- moved on the sheet: C43, C44, C45, C46, C47, C48, C49, C50, C51, C52, C53, C54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

Commit message: finished rough layout
Parts:
- C43, C44, C49, C50, C51, C52, C53, C54: MPN (none) -> CL32B106KBJNNNE
- C45, C46, C47, C48: MPN (none) -> CL05B104KB54PNC
- L1: MPN (none) -> CYA1040-6.8UH
- R25, R29: MPN (none) -> 0402WGF1002TCE
- R26: MPN (none) -> 0402WGF0000TCE
- R27: MPN (none) -> 0402WGF5102TCE
- R28: MPN (none) -> 0402WGF1501TCE
